File: fallout-nametag.kicad_pcb (KiCad board)
At the start: 2 copper layers, 75.4 x 87.9 mm, 30 parts, among them J1 Conn_01x06_Pin, U1 NT3H2111W0FHK, U2 ATtiny85-20S

Commit message: ok i fixed it
Parts:
- added G***: LOGO, LOGO, B.Cu at (136.6, 106.3)
Other:
- board size 75.4 x 87.9 mm -> 79.6 x 92.9 mm
